Commit message: finished environment setup

File: urdf/bouncy.xacro (robot description, xacro)
@@ -1,5 +1,5 @@
 <?xml version="1.0"?>
 <robot name="bouncy" xmlns:xacro="http://www.ros.org/wiki/xacro">
-	<xacro:include filename="/home/oem/ros2_ws/src/bouncy_bot/urdf/bouncy.ign"/>
+    <xacro:include filename="/home/oem/ros2_ws/src/bouncy_bot/urdf/bouncy.ign"/>
     <!-- Parameters -->
     <xacro:property name="ball_mass" value="0.5" />
@@ -10,10 +10,9 @@
     <xacro:property name="enginZpose" value="-0.0408" />
   <link name="outer_ball">
-  	<pose frame="">0 0 0 0 0 0</pose>
     <inertial>
         <mass value="${ball_mass}" />
         <inertia ixx="0.064" ixy="0" ixz="0" iyy="0.064" iyz="0" izz="0.064" />
     </inertial>
-	<collision>
+    <collision>
         <geometry>
             <sphere radius="0.44" />
@@ -22,17 +21,17 @@
     <visual>
         <geometry>
-        	<sphere radius="0.44" />
-	    </geometry>
+            <sphere radius="0.44" />
+        </geometry>
     </visual>
   </link>
-		<!-- Joint - rotation_engin / pull_engin -->
-	<joint name="joint_rotation_engin_pull_engin" type="prismatic">
-	    <origin rpy="0 0 0" xyz="0 0 0"/>
-	    <child link="pull_engin" />
-	    <parent link="rotation_engin" />
-	    <axis rpy="0 0 0" xyz="0 0 1" />
-	    <limit upper="0" lower="-0.4" effort="10000" velocity="1000" />
-	</joint>
-	<!-- Link - pull_engin -->
+    <!-- Joint - rotation_engin / pull_engin -->
+    <joint name="joint_rotation_engin_pull_engin" type="prismatic">
+        <origin rpy="0 0 0" xyz="0 0 0"/>
+        <child link="pull_engin" />
+        <parent link="rotation_engin" />
+        <axis rpy="0 0 0" xyz="0 0 1" />
+        <limit upper="0" lower="-0.37" effort="10000" velocity="1000" />
+    </joint>
+    <!-- Link - pull_engin -->
   <link name="pull_engin">
     <inertial>
@@ -40,24 +39,24 @@
         <inertia ixx="0.001" ixy="0" ixz="0" iyy="0.001" iyz="0" izz="0.001" />
     </inertial>
-	<collision name="collision">
+    <collision>
         <geometry>
-            <sphere radius="0.05" />
+            <box size="0.1 0.1 0.1" />
         </geometry>
     </collision>
     <visual>
         <geometry>
-        	<sphere radius="0.05" />
-	    </geometry>
+            <box size="0.1 0.1 0.1" />
+    </geometry>
     </visual>
   </link>
-		<!-- Joint - outer_ball /  rotation engin-->
-	<joint name="joint_outer_ball_rotation_engin"  type="continuous">
-	    <origin rpy="0 0 0" xyz="0 0 0" />
-	    <child link="rotation_engin" />
-	    <parent link="outer_ball" />
-	    <axis rpy="0 0 0" xyz="0 0 1" />
-	    <limit effort="10000" velocity="5" />
-	    <joint_properties damping="1.0" friction="1.0" />
-	</joint>
+    <!-- Joint - outer_ball /  rotation engin-->
+    <joint name="joint_outer_ball_rotation_engin"  type="continuous">
+        <origin rpy="0 0 0" xyz="0 0 0" />
+        <child link="rotation_engin" />
+        <parent link="outer_ball" />
+        <axis rpy="0 0 0" xyz="0 0 1" />
+        <limit effort="10000" velocity="5" />
+        <joint_properties damping="1.0" friction="1.0" />
+    </joint>
     <link name="rotation_engin">
         <inertial>
@@ -68,5 +67,5 @@
         <collision>
             <geometry>
-                <box size="0.08 0.08 0.87" />
+                <box size="0.02 0.02 0.88" />
             </geometry>
         </collision>
@@ -74,67 +73,67 @@
             <geometry>
                 <box size="0.08 0.08 0.87" />
-			</geometry>
+    </geometry>
         </visual>
     </link>
-		<!-- Joint - pull_engin /  rotating_arms-->
-	<joint name="joint_pull_engin_rotating_arm1"  type="continuous">
-	    <origin rpy="${PI} 0 0" xyz="-0.055 0 0" />
-	    <child link="rotating_arm1" />
-	    <parent link="pull_engin" />
-	    <axis rpy="0 0 0" xyz="1 0 0" >
+    <!-- Joint - pull_engin /  rotating_arms-->
+    <joint name="joint_pull_engin_rotating_arm1"  type="continuous">
+        <origin rpy="${PI} 0 0" xyz="-0.055 0 0" />
+        <child link="rotating_arm1" />
+        <parent link="pull_engin" />
+        <axis rpy="0 0 0" xyz="1 0 0" >
           <dynamics>
-			<friction>1</friction>
+    <friction>1</friction>
           </dynamics>
-		</axis>
-	    <limit effort="10000" velocity="100" />
-	</joint>
-	<link name="rotating_arm1">
-	  <inertial>
-	    <mass value="${arm_mass}" />
-	    <origin xyz="-0 0 0.18" rpy="0 0 0" />
-	    <inertia ixx="0.0116" ixy="0" ixz="0" iyy="0.0108" iyz="0" izz="0.000842" />
-	  </inertial>
-	  <collision>
-	    <origin xyz="-0 0 0.18" rpy="0 0 0" />
-	    <geometry>
-	      <box size="0.01 0.1 0.36" />
-	    </geometry>
-	  </collision>
-	  <visual>
-	    <origin xyz="-0 0 0.18" rpy="0 0 0" />
-	    <geometry>
-	      <box size="0.01 0.1 0.36" />
-	    </geometry>
-	  </visual>
-	</link>
-	<joint name="joint_pull_engin_rotating_arm2"  type="continuous">
-	    <origin rpy="${PI} 0 0" xyz="0.055 0 0" />
-	    <child link="rotating_arm2" />
-	    <parent link="pull_engin" />
-	    <axis rpy="0 0 0" xyz="1 0 0" >
+    </axis>
+        <limit effort="10000" velocity="100" />
+    </joint>
+    <link name="rotating_arm1">
+      <inertial>
+        <mass value="${arm_mass}" />
+        <origin xyz="-0 0 0.18" rpy="0 0 0" />
+        <inertia ixx="0.0116" ixy="0" ixz="0" iyy="0.0108" iyz="0" izz="0.000842" />
+      </inertial>
+      <collision>
+        <origin xyz="-0 0 0.18" rpy="0 0 0" />
+        <geometry>
+          <box size="0.01 0.1 0.36" />
+        </geometry>
+      </collision>
+      <visual>
+        <origin xyz="-0 0 0.18" rpy="0 0 0" />
+        <geometry>
+          <box size="0.01 0.1 0.36" />
+        </geometry>
+      </visual>
+    </link>
+    <joint name="joint_pull_engin_rotating_arm2"  type="continuous">
+        <origin rpy="${PI} 0 0" xyz="0.055 0 0" />
+        <child link="rotating_arm2" />
+        <parent link="pull_engin" />
+        <axis rpy="0 0 0" xyz="1 0 0" >
           <dynamics>
-			<friction>1</friction>
+    <friction>1</friction>
           </dynamics>
-		</axis>
-	    <limit effort="10000" velocity="100" />
-	</joint>
-	<link name="rotating_arm2">
-	  <inertial>
-	    <mass value="${arm_mass}" />
-	    <origin xyz="-0 0 0.18" rpy="0 0 0" />
-	    <inertia ixx="0.0116" ixy="0" ixz="0" iyy="0.0108" iyz="0" izz="0.000842" />
-	  </inertial>
-	  <collision>
-	    <origin xyz="-0 0 0.18" rpy="0 0 0" />
-	    <geometry>
-	      <box size="0.01 0.1 0.36" />
-	    </geometry>
-	  </collision>
-	  <visual>
-	    <origin xyz="-0 0 0.18" rpy="0 0 0" />
-	    <geometry>
-	      <box size="0.01 0.1 0.36" />
-	    </geometry>
-	  </visual>
-	</link>
+    </axis>
+        <limit effort="10000" velocity="100" />
+    </joint>
+    <link name="rotating_arm2">
+      <inertial>
+        <mass value="${arm_mass}" />
+        <origin xyz="-0 0 0.18" rpy="0 0 0" />
+        <inertia ixx="0.0116" ixy="0" ixz="0" iyy="0.0108" iyz="0" izz="0.000842" />
+      </inertial>
+      <collision>
+        <origin xyz="-0 0 0.18" rpy="0 0 0" />
+        <geometry>
+          <box size="0.01 0.1 0.36" />
+        </geometry>
+      </collision>
+      <visual>
+        <origin xyz="-0 0 0.18" rpy="0 0 0" />
+        <geometry>
+          <box size="0.01 0.1 0.36" />
+        </geometry>
+      </visual>
+    </link>
 </robot>
